Commit message: Split Gazebo plugins into moma.gazebo.xacro

File: moma_description/urdf/moma.urdf.xacro (robot description, xacro)
@@ -55,7 +55,4 @@
     </inertial>
   </link>
-  <gazebo reference="mount_box_link">
-    <material>Gazebo/DarkGrey</material>
-  </gazebo>
   <!-- ========================================== -->
   <!-- 3. INCLUDE & INSTANTIATE THE UR ARM        -->
@@ -80,21 +77,6 @@
   </xacro:ur_robot>
   <!-- ========================================== -->
-  <!-- 4. GAZEBO PLUGINS                          -->
+  <!-- 4. GAZEBO                                  -->
   <!-- ========================================== -->
-  <xacro:if value="$(arg sim_ignition)">
-    <gazebo>
-      <plugin filename="ign_ros2_control-system"
-              name="ign_ros2_control::IgnitionROS2ControlPlugin">
-        <parameters>$(find moma_moveit_config)/config/ros2_controllers.yaml</parameters>
-      </plugin>
-      <!-- Ground-truth-physics odometry — replaces diff_drive's lying /odom under wall contact. -->
-      <plugin filename="ignition-gazebo-odometry-publisher-system"
-              name="ignition::gazebo::systems::OdometryPublisher">
-        <odom_frame>odom</odom_frame>
-        <robot_base_frame>base_footprint</robot_base_frame>
-        <odom_topic>odom_gt</odom_topic>
-        <dimensions>2</dimensions>
-      </plugin>
-    </gazebo>
-  </xacro:if>
+  <xacro:include filename="$(find moma_description)/urdf/moma.gazebo.xacro" />
 </robot>
